File: mp1/KiCad/mp1.kicad_pcb (KiCad board)
At the start: 2 copper layers, 17.5 x 14.5 mm, 16 parts, among them J1 480370001, U2 MCP6022-I/ST, U3 MCP1702T-3302E/MB

Commit message: mp1 all files
Other:
- board size 17.5 x 14.5 mm -> 17.5 x 15 mm
Changed lines of the file:
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@@
 	)
 	(gr_line
-		(start 128.5 77.5)
-		(end 146 77.5)
+		(start 128.5 77)
+		(end 146 77)
 		(stroke
 			(width 0.05)
@@
 	(gr_line
 		(start 128.5 92)
-		(end 128.5 77.5)
+		(end 128.5 77)
 		(stroke
 			(width 0.05)
@@
 	)
 	(gr_line
-		(start 146 77.5)
+		(start 146 77)
 		(end 146 92)
 		(stroke
@@
 		(polygon
 			(pts
-				(xy 128.5 77.5) (xy 146 77.5) (xy 146 92) (xy 128.5 92)
+				(xy 128.5 77) (xy 146 77) (xy 146 92) (xy 128.5 92)
 			)
 		)
@@
 		(polygon
 			(pts
-				(xy 128.5 77.5) (xy 146 77.5) (xy 146 92) (xy 128.5 92)
+				(xy 128.5 77) (xy 146 77) (xy 146 92) (xy 128.5 92)
 			)
 		)
